File: bug-pad.kicad_pcb (KiCad board)
At the start: 2 copper layers, 117.5 x 80 mm, 9 parts, among them SW1 SW_Push, SW2 SW_Push, SW3 SW_Push, SW4 SW_Push, SW5 RotaryEncoder_Switch, U1 MOUDLE-SEEEDUINO-XIAO, U2 ER_OLEDM0.91_1x-I2C

Commit message: added all the 3d components cad
Parts:
- added G***: LOGO, demo.preety:github-logo, F.Cu at (200.9, 143.3)
- moved U1 3.43 mm to (126.2, 86.4)
Routing:
- net Net-(U1-PA10_A2_D2): track 65.8 -> 73.9 mm
- net Net-(U1-PA02_A0_D0): track 46.3 -> 51.8 mm
- net Net-(U1-GND): track 244.0 -> 248.3 mm
- net Net-(U1-PB08_A6_D6_TX): track 97.6 -> 101.3 mm
- net Net-(U1-PA11_A3_D3): track 135.5 -> 132.6 mm
- net Net-(U1-PA7_A8_D8_SCK): track 88.4 -> 91.2 mm
- net Net-(U1-3V3): track 10.5 -> 13.2 mm
- net Net-(U1-PA8_A4_D4_SDA): track 32.7 -> 35.1 mm
- net Net-(U1-PA9_A5_D5_SCL): track 34.3 -> 36.7 mm
Other:
- board text added: "ayush-bug"

Commit message: added interactive images on pcb
Parts:
- added G***: LOGO, demo.preety:heisenberg, F.Cu at (199.2, 114.1)
- added G***: LOGO, demo.preety:hackclub-flag-left, F.Cu at (118.4, 118.9)
- added G***: LOGO, demo.preety:hackclub-flag-left, B.Cu at (199.2, 140.7)
- added G***: LOGO, demo.preety:stardance-logo, B.Cu at (186.2, 109.7)
- added G***: LOGO, demo.preety:bug-butterfly, B.Cu at (120.9, 119.4)
Other:
- board text added: "https://github.com/ayush-bug"
